Commit message: Modified launch file for visualising the robot
- The robot now moves in rviz in response to velocities published
  on cmd_vel

File: nuturtle_description/urdf/diff_drive.urdf.xacro (robot description, xacro)
@@ -53,5 +53,5 @@
     </visual>
   </link>
-   <joint name="castor_axle" type="continuous">
+   <joint name="castor_axle" type="fixed">
     <parent link="base_link"/>
     <child link="castor"/>

Commit message: Completed adding inertial properties of the links

File: nuturtle_description/urdf/diff_drive.urdf.xacro (robot description, xacro)
@@ -2,4 +2,5 @@
 <robot xmlns:xacro="http://www.ros.org/wiki/xacro" name="differential_drive_robot">
   <xacro:property name="robot_specs" value="${load_yaml('$(find nuturtle_description)/config/diff_params.yaml')}"/>
+  <xacro:include filename="$(find nuturtle_description)/urdf/inertia_tensor.macro.xacro"/>
   <material name="blue">
     <color rgba="0 0 1 0.5"/>
@@ -14,4 +15,10 @@
     <color rgba="0 0 0 0.0"/>
   </material>
+  <link name="dummy">
+  </link>
+  <joint name="dummy_joint" type="fixed">
+  <parent link="dummy"/>
+  <child link="base_link"/>
+  </joint>
   <link name="base_link">
     <visual>
@@ -22,9 +29,22 @@
       <material name="red"/>
     </visual>
+    <inertial>
+      <origin xyz="-${robot_specs['chasis_length']/2}  0 0" rpy="0 0 0"/>
+      <mass value="${robot_specs['turtle_bot_weight'] - 2 * robot_specs['wheel_weight']}"/>
+      <xacro:box_inertia m="${robot_specs['turtle_bot_weight'] - 2 * robot_specs['wheel_weight']}"
+        x="${robot_specs['chasis_length']}" y="${robot_specs['wheel_base'] - 2 * robot_specs['wheel_width']}"
+        z="${robot_specs['chasis_thickness']}"/>
+    </inertial>
+    <collision>
+      <geometry>
+        <box size="${robot_specs['chasis_length']} ${robot_specs['wheel_base'] - 2 * robot_specs['wheel_width']} ${robot_specs['chasis_thickness']}"/>
+      </geometry>
+      <origin xyz="${robot_specs['chasis_length']/2} 0 0" rpy="0 0 0"/>
+    </collision>
   </link>
    <joint name="left_wheel_axle" type="continuous">
     <parent link="base_link"/>
     <child link="left_wheel"/>
-    <origin xyz="0  ${(robot_specs['wheel_base'] - 2 * robot_specs['wheel_width'])/2} 0"/>
+    <origin xyz="0  ${(robot_specs['wheel_base'] - 2 * robot_specs['wheel_width'])/2} ${(-robot_specs['chasis_thickness']/2.0+robot_specs['wheel_axle_offset'])}"/>
     <axis xyz="0 1 0"/>
    </joint>
@@ -37,9 +57,28 @@
       <material name="black"/>
     </visual>
+    <inertial>
+      <origin xyz="0 ${robot_specs['wheel_width']/2}  0" rpy="0 ${-pi/2} 0"/>
+      <mass value="${robot_specs['wheel_weight']}"/>
+      <xacro:cylinder_inertia m="${robot_specs['wheel_weight']}"
+        r="${robot_specs['wheel_radius']}" h="${robot_specs['wheel_width']}"/>
+    </inertial>
+    <collision>
+      <geometry>
+        <cylinder length="${robot_specs['wheel_width']}" radius="${robot_specs['wheel_radius']}"/>
+      </geometry>
+      <origin xyz="0 ${robot_specs['wheel_width']/2} 0" rpy="${-pi/2.0} 0 0"/>
+    </collision>
   </link>
+   <joint name="scan_link_joint" type="fixed">
+    <parent link="base_link"/>
+    <child link="base_scan"/>
+    <origin xyz="0 0 ${robot_specs['chasis_thickness']/2}"/>
+   </joint>
+   <link name="base_scan">
+   </link>
    <joint name="right_wheel_axle" type="continuous">
     <parent link="base_link"/>
     <child link="right_wheel"/>
-    <origin xyz="0  ${-(robot_specs['wheel_base'] - 2 * robot_specs['wheel_width'])/2} 0"/>
+    <origin xyz="0  ${-(robot_specs['wheel_base'] - 2 * robot_specs['wheel_width'])/2} ${(-robot_specs['chasis_thickness']/2.0+robot_specs['wheel_axle_offset'])}"/>
     <axis xyz="0 1 0"/>
    </joint>
@@ -52,4 +91,16 @@
       <material name="black"/>
     </visual>
+    <inertial>
+      <origin xyz="0 ${-robot_specs['wheel_width']/2}  0" rpy="0 ${-pi/2} 0"/>
+      <mass value="${robot_specs['wheel_weight']}"/>
+      <xacro:cylinder_inertia m="${robot_specs['wheel_weight']}"
+        r="${robot_specs['wheel_radius']}" h="${robot_specs['wheel_width']}"/>
+    </inertial>
+    <collision>
+      <geometry>
+        <cylinder length="${robot_specs['wheel_width']}" radius="${robot_specs['wheel_radius']}"/>
+      </geometry>
+      <origin xyz="0 ${-robot_specs['wheel_width']/2} 0" rpy="${-pi/2.0} 0 0"/>
+    </collision>
   </link>
    <joint name="castor_axle" type="fixed">
@@ -67,4 +118,10 @@
       <material name="black"/>
     </visual>
+    <collision>
+      <geometry>
+        <sphere radius="${robot_specs['wheel_radius']/4}"/>
+      </geometry>
+      <origin xyz="0 0 0" rpy="0 0 0"/>
+    </collision>
   </link>
 </robot>

Commit message: Added gazebo tags to the turtlebot model and launched in gazebo

File: nuturtle_description/urdf/diff_drive.urdf.xacro (robot description, xacro)
@@ -15,10 +15,10 @@
     <color rgba="0 0 0 0.0"/>
   </material>
-  <link name="dummy">
+  <!-- link name="dummy">
   </link>
   <joint name="dummy_joint" type="fixed">
   <parent link="dummy"/>
   <child link="base_link"/>
-  </joint>
+  </joint -->
   <link name="base_link">
     <visual>
@@ -30,9 +30,12 @@
     </visual>
     <inertial>
-      <origin xyz="-${robot_specs['chasis_length']/2}  0 0" rpy="0 0 0"/>
+      <origin xyz="${robot_specs['chasis_length']/2}  0 0" rpy="0 0 0"/>
       <mass value="${robot_specs['turtle_bot_weight'] - 2 * robot_specs['wheel_weight']}"/>
       <xacro:box_inertia m="${robot_specs['turtle_bot_weight'] - 2 * robot_specs['wheel_weight']}"
         x="${robot_specs['chasis_length']}" y="${robot_specs['wheel_base'] - 2 * robot_specs['wheel_width']}"
         z="${robot_specs['chasis_thickness']}"/>
+      <!-- inertia  ixx="100000.0" ixy = "0" ixz = "0"
+                  iyy="100000.0" iyz = "0"
+                  izz="100000.0"/ -->
     </inertial>
     <collision>
@@ -62,4 +65,7 @@
       <xacro:cylinder_inertia m="${robot_specs['wheel_weight']}"
         r="${robot_specs['wheel_radius']}" h="${robot_specs['wheel_width']}"/>
+      <!--inertia  ixx="1.0" ixy = "0" ixz = "0"
+                  iyy="1.0" iyz = "0"
+                  izz="1.0" /-->
     </inertial>
     <collision>
@@ -96,4 +102,7 @@
       <xacro:cylinder_inertia m="${robot_specs['wheel_weight']}"
         r="${robot_specs['wheel_radius']}" h="${robot_specs['wheel_width']}"/>
+      <!-- inertia  ixx="1.0" ixy = "0" ixz = "0"
+                  iyy="1.0" iyz = "0"
+                  izz="1.0" / -->
     </inertial>
     <collision>
@@ -124,4 +133,10 @@
       <origin xyz="0 0 0" rpy="0 0 0"/>
     </collision>
+    <inertial>
+      <mass value="0"/>
+      <inertia  ixx="0.0" ixy = "0" ixz = "0"
+                  iyy="0.0" iyz = "0"
+                  izz="0.0" />
+    </inertial>
   </link>
 </robot>

Commit message: Refined inertial tags for accurate robot visualisation in gazebo

File: nuturtle_description/urdf/diff_drive.urdf.xacro (robot description, xacro)
@@ -15,10 +15,10 @@
     <color rgba="0 0 0 0.0"/>
   </material>
-  <!-- link name="dummy">
+  <link name="dummy">
   </link>
   <joint name="dummy_joint" type="fixed">
   <parent link="dummy"/>
   <child link="base_link"/>
-  </joint -->
+  </joint>
   <link name="base_link">
     <visual>
@@ -61,5 +61,5 @@
     </visual>
     <inertial>
-      <origin xyz="0 ${robot_specs['wheel_width']/2}  0" rpy="0 ${-pi/2} 0"/>
+      <origin xyz="0 ${robot_specs['wheel_width']/2} 0" rpy="${-pi/2.0} 0 0"/>
       <mass value="${robot_specs['wheel_weight']}"/>
       <xacro:cylinder_inertia m="${robot_specs['wheel_weight']}"
@@ -98,5 +98,6 @@
     </visual>
     <inertial>
-      <origin xyz="0 ${-robot_specs['wheel_width']/2}  0" rpy="0 ${-pi/2} 0"/>
+      <origin xyz="0 ${-robot_specs['wheel_width']/2} 0" rpy="${-pi/2.0} 0 0"/>
+      <material name="black"/>
       <mass value="${robot_specs['wheel_weight']}"/>
       <xacro:cylinder_inertia m="${robot_specs['wheel_weight']}"

Commit message: Started the basic skeleton of the EKF algorithm
- Integrated odometry into the pipeline

File: nuturtle_description/urdf/diff_drive.urdf.xacro (robot description, xacro)
@@ -15,11 +15,13 @@
     <color rgba="0 0 0 0.0"/>
   </material>
-  <link name="dummy">
+  <link name="base_link">
   </link>
-  <joint name="dummy_joint" type="fixed">
-  <parent link="dummy"/>
-  <child link="base_link"/>
+  <joint name="base_link_joint" type="fixed">
+  <parent link="base_link"/>
+  <child link="robot_link"/>
+  <origin xyz="0 0 0"/>
+  <axis xyz="0 0 0"/>
   </joint>
-  <link name="base_link">
+  <link name="robot_link">
     <visual>
       <geometry>
@@ -47,5 +49,5 @@
   </link>
    <joint name="left_wheel_axle" type="continuous">
-    <parent link="base_link"/>
+    <parent link="robot_link"/>
     <child link="left_wheel"/>
     <origin xyz="0  ${(robot_specs['wheel_base'] - 2 * robot_specs['wheel_width'])/2} ${(-robot_specs['chasis_thickness']/2.0+robot_specs['wheel_axle_offset'])}"/>
@@ -77,5 +79,5 @@
   </link>
    <joint name="scan_link_joint" type="fixed">
-    <parent link="base_link"/>
+    <parent link="robot_link"/>
     <child link="base_scan"/>
     <origin xyz="0 0 ${robot_specs['chasis_thickness']/2}"/>
@@ -84,5 +86,5 @@
    </link>
    <joint name="right_wheel_axle" type="continuous">
-    <parent link="base_link"/>
+    <parent link="robot_link"/>
     <child link="right_wheel"/>
     <origin xyz="0  ${-(robot_specs['wheel_base'] - 2 * robot_specs['wheel_width'])/2} ${(-robot_specs['chasis_thickness']/2.0+robot_specs['wheel_axle_offset'])}"/>
@@ -115,5 +117,5 @@
   </link>
    <joint name="castor_axle" type="fixed">
-    <parent link="base_link"/>
+    <parent link="robot_link"/>
     <child link="castor"/>
     <origin xyz="${robot_specs['chasis_length'] - robot_specs['wheel_radius']/4} 0 ${-robot_specs['chasis_thickness']/2-robot_specs['wheel_radius']/4}"/>

Commit message: Added a launch file for known data association - the basic launch file will run analysis node for landmark detection   when run with debug=true

File: nuturtle_description/urdf/diff_drive.urdf.xacro (robot description, xacro)
@@ -81,5 +81,5 @@
     <parent link="robot_link"/>
     <child link="base_scan"/>
-    <origin xyz="0 0 ${robot_specs['chasis_thickness']/2}"/>
+    <origin xyz="0 0 ${robot_specs['chasis_thickness']/2+0.01}"/>
    </joint>
    <link name="base_scan">
